File: Huellas_Circuito/kikad_2/proyecto1/proyecto1/proyecto1.kicad_sch (KiCad schematic)
At the start: 9 parts, among them SW1 SW_DIP_x01, U1 ESP32-DEVKIT-V1

Commit message: Creacion_Footprint_Regul&Conectado
Parts:
- removed SW1: SW_DIP_x01, symbol Switch:SW_DIP_x01
- added S1: OS102011MS2QN1, OS102011MS2QN1:SW_OS102011MS2QN1, symbol OS102011MS2QN1:OS102011MS2QN1
- D1: footprint (none) -> LED_THT:LED_D3.0mm
- RGUL1: footprint (none) -> Regulador:RGUL1
- renumbered Moto1 to Motor1
Connections:
- net GND: now also S1.1
- net VDRV: now also S1.2
- net at Bateria1.1 (Pin_1): now also S1.3
- net VIN renamed Vin
